Commit message: ptz camera tracking the drone 	-camera view centered

File: src/drone_detector/robot_description/fixed_lidar.xacro (robot description, xacro)
@@ -49,7 +49,8 @@
     <origin xyz="0 0 3.0" rpy="0 0 0"/>
   </joint>
-  <!-- Attach PTZ Camera on top of LiDAR -->
-  <xacro:ptz_camera parent_link="fixed_lidar">
-    <origin xyz="0 0 0.15" rpy="0 0 0"/>
+  <!-- PTZ camera is on a separate pole 1.25 m beside the LiDAR pole.
+       Its top is at z=3.4 m, slightly above the 3.0 m LiDAR stand. -->
+  <xacro:ptz_camera parent_link="base_link">
+    <origin xyz="0.6 0 3.4" rpy="0 0 0"/>
   </xacro:ptz_camera>
 </robot>

File: src/drone_detector/robot_description/ptz_camera.xacro (robot description, xacro)
@@ -4,4 +4,13 @@
     <!-- Camera Base Link -->
     <link name="camera_base_link">
+      <visual name="support_pole_visual">
+        <origin xyz="0 0 -1.70" rpy="0 0 0"/>
+        <geometry>
+          <cylinder radius="0.05" length="3.40"/>
+        </geometry>
+        <material name="support_pole_material">
+          <color rgba="0.55 0.55 0.55 1.0"/>
+        </material>
+      </visual>
       <visual>
         <origin xyz="0 0 0.10" rpy="0 0 0"/>
@@ -23,5 +32,6 @@
     <link name="pan_link">
       <visual>
-        <origin xyz="0 0 0.15" rpy="0 0 0"/>
+        <!-- Seat the pan cylinder directly on the camera base. -->
+        <origin xyz="0 0 0.05" rpy="0 0 0"/>
         <geometry>
           <cylinder radius="0.22" length="0.10"/>
@@ -59,5 +69,5 @@
       <parent link="pan_link"/>
       <child link="tilt_link"/>
-      <origin xyz="0 0 0.20" rpy="0 0 0"/>
+      <origin xyz="0 0 0.10" rpy="0 0 0"/>
       <axis xyz="0 1 0"/>
       <limit lower="-1.0472" upper="1.0472" effort="10" velocity="1.0"/>
